File: chunair/chunair/chunair_v2/chunair.kicad_pcb (KiCad board)
At the start: 2 copper layers, 218.6 x 37.6 mm, 19 parts, among them J1 Conn_01x08_Male, J2 Conn_01x08_Male

Commit message: v2.0 | Added first ordered revision of PCBs
Parts:
- added G***: LOGO, chunair_local:logo_small, B.Cu at (242.0, 99.0)
- added G***: LOGO, chunair_local:logo_small, F.Cu at (242.0, 99.0)
