File: chunair/chunair_core/chunair_core.kicad_pcb (KiCad board)
At the start: 2 copper layers, 34 x 52 mm, 7 parts, among them J1 Conn_01x08_Male, J2 Conn_01x08_Male, J3 Conn_01x03_Male, U1 ProMicro

Commit message: v2.0 | Added first ordered revision of PCBs
Parts:
- added G***: LOGO, chunair_local:logo, B.Cu at (150.0, 69.0)
- moved J1 24.0 mm to (138.0, 89.0)
- moved J2 24.0 mm to (162.0, 89.0)
Routing:
- net /8: track 54.8 -> 13.7 mm, vias 1 -> 0
- net /A10: track 16.5 -> 47.8 mm
- net /coin: track 68.4 -> 41.4 mm
- net /6: track 41.9 -> 16.8 mm, vias 1 -> 0
- net /RGB_R: track 64.4 -> 45.2 mm
- net /A1: track 32.2 -> 49.7 mm
- net /16: track 34.0 -> 17.0 mm, vias 1 -> 0
- net GND: track 100.1 -> 84.0 mm, vias 0 -> 2
- net /A3: track 39.7 -> 55.7 mm
- net /A0: track 46.9 -> 32.5 mm, vias 1 -> 0
- net /7: track 13.5 -> 24.2 mm
- net /A2: track 50.5 -> 40.5 mm
- net /A9: track 16.0 -> 25.6 mm
- net /14: track 17.0 -> 25.9 mm, vias 0 -> 1
- net +5V: track 64.9 -> 59.5 mm, vias 0 -> 2
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Other:
- board size 34 x 52 mm -> 34 x 53 mm
- board text added: "JLCJLCJLCJLC"
